File: hybrid_pmod_v2.kicad_pcb (KiCad board)
At the start: 4 copper layers, 64.3 x 22.9 mm, 28 parts, among them J1 I2C Connector, J2 I2C Connector, J3 HDMI_A, J4 Ground Pin, J5 Power Input, U1 DS25CP102TSQ/NOPB, U2 DS25CP102TSQ/NOPB, U3 P82B715

Commit message: Many changes, suggestions from H. T. Johansson.
Parts:
- added C10: 1u, Capacitor_SMD:C_0402_1005Metric_Pad0.74x0.62mm_HandSolder, F.Cu at (104.4, 68.0)
- added C7: 1u, Capacitor_SMD:C_0402_1005Metric_Pad0.74x0.62mm_HandSolder, F.Cu at (104.4, 86.9)
- added C8: 100n, Capacitor_SMD:C_0402_1005Metric_Pad0.74x0.62mm_HandSolder, F.Cu at (103.4, 86.9)
- added C9: 100n, Capacitor_SMD:C_0402_1005Metric_Pad0.74x0.62mm_HandSolder, F.Cu at (103.4, 68.0)
- C1, C2, C3, C4, C5, C6: footprint Capacitor_SMD:C_0603_1608Metric_Pad1.08x0.95mm_HandSolder -> Capacitor_SMD:C_0402_1005Metric_Pad0.74x0.62mm_HandSolder
- R1, R10, R11, R12, R2, R3, R4, R5, R6, R7, R8, R9: footprint Resistor_SMD:R_0603_1608Metric_Pad0.98x0.95mm_HandSolder -> Resistor_SMD:R_0402_1005Metric_Pad0.72x0.64mm_HandSolder
- moved R11 1.59 mm to (99.3, 87.0)
- moved R8 1.54 mm to (102.4, 86.9)
- moved R3 1.44 mm to (102.4, 68.0)
- moved R9 1.05 mm to (101.3, 86.9)
- moved R5 0.95 mm to (101.3, 68.0)
- moved R12 0.93 mm to (100.3, 87.0)
- moved R6 0.47 mm to (100.3, 68.0)
Routing:
- net /CLOCK_P: track 34.3 -> 32.2 mm
- net +3.3V: track 35.6 -> 37.1 mm
- net /CONTROL_P: track 27.2 -> 28.5 mm
- net /CLOCK_N: track 27.9 -> 28.8 mm
- net GND: track 41.0 -> 41.6 mm, vias 16 -> 47
- net /DATA1_N: track 25.7 -> 25.2 mm
Other:
- board text added: "+3.3V"
- board text added: "GND"
- board text added: "IN"
- board text added: "OUT"
