File: hybrid_pmod_v2.kicad_sch (KiCad schematic)
At the start: 28 parts, among them J1 I2C Connector, J2 I2C Connector, J3 HDMI_A, J4 Ground Pin, J5 Power Input, U1 DS25CP102TSQ/NOPB, U2 DS25CP102TSQ/NOPB, U3 P82B715

Commit message: Many changes, suggestions from H. T. Johansson.
Parts:
- added C10, C7: 1u, Capacitor_SMD:C_0402_1005Metric_Pad0.74x0.62mm_HandSolder, symbol Device:C
- added C8, C9: 100n, Capacitor_SMD:C_0402_1005Metric_Pad0.74x0.62mm_HandSolder, symbol Device:C
- C1, C2, C3, C4, C5, C6: footprint Capacitor_SMD:C_0603_1608Metric_Pad1.08x0.95mm_HandSolder -> Capacitor_SMD:C_0402_1005Metric_Pad0.74x0.62mm_HandSolder
- R1, R10, R11, R12, R2, R3, R4, R5, R6, R7, R8, R9: footprint Resistor_SMD:R_0603_1608Metric_Pad0.98x0.95mm_HandSolder -> Resistor_SMD:R_0402_1005Metric_Pad0.72x0.64mm_HandSolder
Connections:
- net GND: now also C10.2, C7.2, C8.2, C9.2
- net at JP1.1 (A), R11.1, R12.1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: now also C10.1, C7.1, C8.1, C9.1
Other:
- note added: "Pull-Up resistors for TMDS"
- moved on the sheet: J4, J5, JP1, R1, R11, R12, R2, R3, R5, R6, R7, R8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
